Commit message: fixed: dh params

File: lab_2/urdf/dynamicmodel.urdf.xacro (robot description, xacro)
@@ -1,6 +1,12 @@
 <?xml version="1.0"?>
 <robot name="robot" xmlns:xacro="http://www.ros.org/wiki/xacro">
-    <xacro:property name="parameters" value="${load_yaml('..//yaml/urdf.yaml')}"/>
-    <xacro:property name="sizeparams" value="${load_yaml('..//yaml/sizeparams.yaml')}"/>
+    <xacro:property name="props" value="${load_yaml('..//yaml/urdf.yaml')}"/>
+    <xacro:property name="size" value="${load_yaml('..//yaml/sizeparams.yaml')}"/>
+    <material name="red">
+        <color rgba="1 0.0 0.0 1"/>
+    </material>
+    <material name="green">
+        <color rgba="0.0 1.0 0.0 1.0"/>
+    </material>
     <material name="blue">
         <color rgba="0 0 1 1"/>
@@ -9,63 +15,60 @@
         <color rgba="1 1 1 1"/>
     </material>
-    <material name="red">
-        <color rgba="1 0 0 1"/>
-    </material>
-   <material name="green">
-        <color rgba="0 1 0 1"/>
-   </material>
     <link name="base_link">
         <visual>
             <geometry>
-                <cylinder length="${sizeparams['base_height']}" radius="${sizeparams['base_width']}"/>
+                <cylinder length="${size['base_height']}" radius="${size['base_width']}"/>
             </geometry>
-            <origin xyz="0 0 ${sizeparams['base_height']/2}"/>
+            <origin xyz="0 0 0"/>
+            <material name="blue"/>
+        </visual>
+    </link>
+    <link name="link_1">
+        <visual>
+            <geometry>
+                <box size="${size['linki1_width']} ${size['linki1_width']} ${props['i2']['l_len']}"/>
+            </geometry>
+            <origin xyz="${props['i2']['l_xyz']}" rpy="${props['i2']['l_rpy']}"/>
+            <material name="red"/>
+        </visual>
+    </link>
+    <link name="link_2">
+        <visual>
+            <geometry>
+                <box size="${size['linki2_width']} ${size['linki2_width']} ${props['i3']['l_len']}"/>
+            </geometry>
+            <origin xyz="${props['i3']['l_xyz']}" rpy="${props['i3']['l_rpy']}"/>
+            <material name="green"/>
+        </visual>
+    </link>
+    <link name="link_3">
+        <visual>
+            <geometry>
+                <box size="${size['linki3_width']} ${size['linki3_width']} ${size['linki3_height']}"/>
+            </geometry>
+            <origin xyz="0 0 0" rpy="0 0 0"/>
             <material name="white"/>
         </visual>
     </link>
-    <link name="link1">
-        <visual>
-            <geometry>
-                <box size="${sizeparams['linki1_height']} ${sizeparams['linki1_width']} ${sizeparams['linki1_width']}"/>
-            </geometry>
-            <origin xyz="${parameters['i1']['l_xyz']}" rpy="${parameters['i1']['l_rpy']}"/>
-            <material name="blue"/>
-        </visual>
-    </link>
-    <link name="link2">
-        <visual>
-            <geometry>
-                <box size="${sizeparams['linki2_height']} ${sizeparams['linki2_width']} ${sizeparams['linki2_width']} "/>
-            </geometry>
-            <origin xyz="${parameters['i2']['l_xyz']}" rpy="${parameters['i2']['l_rpy']}"/>
-            <material name="green"/>
-        </visual>
-    </link>
-    <link name="link3">
-        <visual>
-            <geometry>
-                <box size="${sizeparams['linki3_height']} ${sizeparams['linki3_width']} ${sizeparams['linki3_width']}"/>
-            </geometry>
-            <origin xyz="${sizeparams['linki3_height']/2} 0 0" rpy="0 0 0"/>
-            <material name="red"/>
-        </visual>
-    </link>
-    <joint name="base_link1" type="continuous">
+    <joint name="base_link1" type="prismatic">
         <parent link="base_link"/>
-        <child link="link1"/>
-        <origin xyz="0 0 ${sizeparams['base_height']}" rpy="0 0 0"/>
+        <child link="link_1"/>
+        <origin xyz="${props['i1']['j_xyz']}" rpy="${props['i1']['j_rpy']}"/>
+        <axis xyz="0 0 1"/>
+        <limit effort="1000.0" lower="-0.4" upper="0" velocity="0.5"/>
+    </joint>
+    <joint name="link1_link2" type="prismatic">
+        <parent link="link_1"/>
+        <child link="link_2"/>
+        <origin xyz="${props['i2']['j_xyz']}" rpy="${props['i2']['j_rpy']}"/>
+        <axis xyz="0 0 1"/>
+        <limit effort="1000.0" lower="-0.4" upper="0" velocity="0.5"/>
+    </joint>
+    <joint name="link2_link3" type="prismatic">
+        <parent link="link_2"/>
+        <child link="link_3"/>
+        <origin xyz="${props['i3']['j_xyz']}" rpy="${props['i3']['j_rpy']}"/>
+        <limit effort="1000.0" lower="-0.1" upper="0.1" velocity="0.5"/>
         <axis xyz="0 0 1"/>
     </joint>
-    <joint name="link1_link2" type="continuous">
-        <parent link="link1"/>
-        <child link="link2"/>
-        <origin xyz="${parameters['i1']['j_xyz']}" rpy="${parameters['i1']['j_rpy']}"/>
-        <axis xyz="0 0 1"/>
-    </joint>
-    <joint name="link2_link3" type="continuous">
-        <parent link="link2"/>
-        <child link="link3"/>
-        <origin xyz="${parameters['i2']['j_xyz']}" rpy="${parameters['i2']['j_rpy']}"/>
-        <axis xyz="0 1 0"/>
-    </joint>
 </robot>

File: lab_2/urdf/staticmodel.urdf.xacro (robot description, xacro)
@@ -1,6 +1,12 @@
 <?xml version="1.0"?>
 <robot name="robot" xmlns:xacro="http://www.ros.org/wiki/xacro">
-    <xacro:property name="parameters" value="${load_yaml('..//yaml/urdf.yaml')}"/>
-    <xacro:property name="sizeparams" value="${load_yaml('..//yaml/sizeparams.yaml')}"/>
+    <xacro:property name="props" value="${load_yaml('..//yaml/urdf.yaml')}"/>
+    <xacro:property name="size" value="${load_yaml('..//yaml/sizeparams.yaml')}"/>
+    <material name="red">
+        <color rgba="1 0.0 0.0 1"/>
+    </material>
+    <material name="green">
+        <color rgba="0.0 1.0 0.0 1.0"/>
+    </material>
     <material name="blue">
         <color rgba="0 0 1 1"/>
@@ -9,63 +15,57 @@
         <color rgba="1 1 1 1"/>
     </material>
-    <material name="red">
-        <color rgba="1 0 0 1"/>
-    </material>
-   <material name="green">
-        <color rgba="0 1 0 1"/>
-   </material>
     <link name="base_link">
         <visual>
             <geometry>
-                <cylinder length="${sizeparams['base_height']}" radius="${sizeparams['base_width']}"/>
+                <cylinder length="${size['base_height']}" radius="${size['base_width']}"/>
             </geometry>
-            <origin xyz="0 0 ${sizeparams['base_height']/2}"/>
-            <material name="white"/>
-        </visual>
-    </link>
-    <link name="link1">
-        <visual>
-            <geometry>
-                <box size="${sizeparams['linki1_height']} ${sizeparams['linki1_width']} ${sizeparams['linki1_width']}"/>
-            </geometry>
-            <origin xyz="${parameters['i1']['l_xyz']}" rpy="${parameters['i1']['l_rpy']}"/>
+            <origin xyz="0 0 0"/>
             <material name="blue"/>
         </visual>
     </link>
-    <link name="link2">
+    <link name="link_1">
         <visual>
             <geometry>
-                <box size="${sizeparams['linki2_height']} ${sizeparams['linki2_width']} ${sizeparams['linki2_width']} "/>
+                <box size="${size['linki1_width']} ${size['linki1_width']} ${props['i2']['l_len']}"/>
             </geometry>
-            <origin xyz="${parameters['i2']['l_xyz']}" rpy="${parameters['i2']['l_rpy']}"/>
+            <origin xyz="${props['i2']['l_xyz']}" rpy="${props['i2']['l_rpy']}"/>
+            <material name="red"/>
+        </visual>
+    </link>
+    <link name="link_2">
+        <visual>
+            <geometry>
+                <box size="${size['linki2_width']} ${size['linki2_width']} ${props['i3']['l_len']}"/>
+            </geometry>
+            <origin xyz="${props['i3']['l_xyz']}" rpy="${props['i3']['l_rpy']}"/>
             <material name="green"/>
         </visual>
     </link>
-    <link name="link3">
+    <link name="link_3">
         <visual>
             <geometry>
-                <box size="${sizeparams['linki3_height']} ${sizeparams['linki3_width']} ${sizeparams['linki3_width']}"/>
+                <box size="${size['linki3_width']} ${size['linki3_width']} ${size['linki3_height']}"/>
             </geometry>
-            <origin xyz="${sizeparams['linki3_height']/2} 0 0" rpy="0 0 0"/>
-            <material name="red"/>
+            <origin xyz="0 0 0" rpy="0 0 0"/>
+            <material name="white"/>
         </visual>
     </link>
     <joint name="base_link1" type="fixed">
         <parent link="base_link"/>
-        <child link="link1"/>
-        <origin xyz="0 0 ${sizeparams['base_height']}" rpy="0 0 0"/>
+        <child link="link_1"/>
+        <origin xyz="${props['i1']['j_xyz']}" rpy="${props['i1']['j_rpy']}"/>
         <axis xyz="0 0 1"/>
     </joint>
     <joint name="link1_link2" type="fixed">
-        <parent link="link1"/>
-        <child link="link2"/>
-        <origin xyz="${parameters['i1']['j_xyz']}" rpy="${parameters['i1']['j_rpy']}"/>
+        <parent link="link_1"/>
+        <child link="link_2"/>
+        <origin xyz="${props['i2']['j_xyz']}" rpy="${props['i2']['j_rpy']}"/>
         <axis xyz="0 0 1"/>
     </joint>
     <joint name="link2_link3" type="fixed">
-        <parent link="link2"/>
-        <child link="link3"/>
-        <origin xyz="${parameters['i2']['j_xyz']}" rpy="${parameters['i2']['j_rpy']}"/>
-        <axis xyz="0 1 0"/>
+        <parent link="link_2"/>
+        <child link="link_3"/>
+        <origin xyz="${props['i3']['j_xyz']}" rpy="${props['i3']['j_rpy']}"/>
+        <axis xyz="0 0 1"/>
     </joint>
 </robot>
