Commit message: fixed jint

File: lab2-poprawa/urdf/dynamicmodel.urdf.xacro (robot description, xacro)
@@ -63,5 +63,5 @@
         <origin xyz="${props['i2']['j_xyz']}" rpy="${props['i2']['j_rpy']}"/>
         <axis xyz="0 0 1"/>
-        <limit effort="1000.0" lower="-1.57" upper="1.57" velocity="0.5"/>
+        <limit effort="1000.0" lower="-3.14" upper="3.14" velocity="0.5"/>
     </joint>
     <joint name="link2_link3" type="revolute">
@@ -69,5 +69,5 @@
         <child link="link_3"/>
         <origin xyz="${props['i3']['j_xyz']}" rpy="${props['i3']['j_rpy']}"/>
-        <limit effort="1000.0" lower="-1" upper="1" velocity="0.5"/>
+        <limit effort="1000.0" lower="-1.57" upper="1.57" velocity="0.5"/>
         <axis xyz="0 0 1"/>
     </joint>
